File: FPS 100/Backplane/Backplane.kicad_pcb (KiCad board)
At the start: 4 copper layers, 27 parts

Commit message: 2026/1/6
Parts:
- moved UNIBUS_XFER_J1 190.8 mm to (347.9, 367.7), turned to 90 degrees
Connections:
- 4401_FA_J1 pad 93: A1MBS05* -> A2MBS05*
- 4401_FA_J1 pad 95: A1MBS06* -> A2MBS06*
- 4401_FA_J1 pad 97: A1MBS07* -> A2MBS07*
- 4402_DPR_J2 pad 97: BPMBS16* -> DPMBS16*
Routing:
- net +5V: track 695.6 -> 1476.8 mm
- net DPMBS19*: track 0.00 -> 456.2 mm, vias 0 -> 7
- net DPMBS18*: track 0.00 -> 405.4 mm, vias 0 -> 9
- net FMUL*: track 0.00 -> 404.7 mm, vias 0 -> 4
- net DPMBS17*: track 0.00 -> 404.1 mm, vias 0 -> 6
- net BH2HD: track 0.00 -> 320.8 mm, vias 0 -> 1
- net DPMBS24*: track 0.00 -> 305.2 mm, vias 0 -> 10
- net TM2PNL: track 0.00 -> 304.5 mm, vias 0 -> 1
- net SR2HD*: track 0.00 -> 290.5 mm, vias 0 -> 1
- net TMREGE: track 0.00 -> 270.1 mm, vias 0 -> 1
- net MDWRT3: track 0.00 -> 266.0 mm, vias 0 -> 2
- net IODRDY*: track 0.00 -> 262.9 mm, vias 0 -> 1
- net I+H10: track 0.00 -> 253.6 mm, vias 0 -> 1
- net DPMBS27*: track 0.00 -> 245.5 mm, vias 0 -> 6
- net INT2A1E*: track 0.00 -> 244.9 mm, vias 0 -> 1
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Other:
- copper layers 4 -> 6
